Commit message: Updated robot package and simulation files

File: pet_bot_test5/urdf/pet_bot_test5.urdf.xacro (robot description, xacro)
@@ -1049,25 +1049,128 @@
   </ros2_control>
   <!--camera link sensor-->
-  <gazebo reference="depth_camera">
-    <sensor name="depth_camera" type="depth_camera">
+  <link name="camera_optical_frame">
+    <inertial>
+      <mass value="0.001" />
+      <inertia ixx="0.00001" ixy="0" ixz="0" iyy="0.00001" iyz="0" izz="0.00001" />
+    </inertial>
+  </link>
+  <joint name="camera_optical_joint" type="fixed">
+    <parent link="depth_camera"/>
+    <child link="camera_optical_frame"/>
+    <!-- change here as you adjust camera -->
+    <axis xyz="0 0 1"/>
+    <origin xyz="0 0 0" rpy="0 0.0 0"/>
+  </joint>
+  <gazebo reference="camera_optical_frame">
+      <sensor name="realsense2_camera" type="rgbd_camera">
+        <ignition_frame_id>camera_optical_frame</ignition_frame_id>
+        <camera name="realsense2_camera">
+          <horizontal_fov>1.2043</horizontal_fov>
+          <lens>
+            <intrinsics>
+              <fx>915.3003540039062</fx>
+              <fy>914.0320434570312</fy>
+              <cx>642.724365234375</cx>
+              <cy>361.9780578613281</cy>
+              <s>0</s>
+            </intrinsics>
+          </lens>
+          <distortion>
+            <k1>0.0</k1>
+            <k2>0.0</k2>
+            <k3>0.0</k3>
+            <p1>0.0</p1>
+            <p2>0.0</p2>
+            <center>0.5 0.5</center>
+          </distortion>
+          <image>
+            <width>1280</width>
+            <height>720</height>
+            <format>R8G8B8</format>
+          </image>
+          <clip>
+            <near>0.1</near>
+            <far>100</far>
+          </clip>
+          <depth_camera>
+            <clip>
+              <near>0.1</near>
+              <far>100</far>
+            </clip>
+          </depth_camera>
+          <noise>
+            <type>gaussian</type>
+            <mean>0.0</mean>
+            <stddev>0.007</stddev>
+          </noise>
+        </camera>
+        <always_on>1</always_on>
+        <update_rate>2</update_rate>
+        <visualize>0</visualize>
+        <topic>camera</topic>
+      </sensor>
+  </gazebo>
+<link name="lidar_link">
+    <visual>
+      <geometry>
+        <cylinder radius="0.03" length="0.04"/>
+      </geometry>
+      <material name="black">
+        <color rgba="0.1 0.1 0.1 1"/>
+      </material>
+    </visual>
+    <collision>
+      <geometry>
+        <cylinder radius="0.03" length="0.04"/>
+      </geometry>
+    </collision>
+    <inertial>
+      <mass value="0.01"/>
+      <origin xyz="0 0 0"/>
+      <inertia
+        ixx="0.0001" ixy="0" ixz="0"
+        iyy="0.0001" iyz="0"
+        izz="0.0001"/>
+    </inertial>
+  </link>
+  <joint name="lidar_joint" type="fixed">
+  <parent link="base_link"/>
+  <child link="lidar_link"/>
+  <origin xyz="0 0 0" rpy="0 0 0"/>
+</joint>
+<gazebo reference="lidar_link">
+    <sensor name="laser" type="gpu_lidar">
       <always_on>true</always_on>
+      <visualize>false</visualize>
+      <topic>scan</topic>
+      <pose>0 0 0 0 0 0</pose>
       <update_rate>10</update_rate>
-      <visualize>true</visualize>
-      <camera>
-        <horizontal_fov>1.047</horizontal_fov>
-        <image>
-          <width>640</width>
-          <height>480</height>
-          <!-- <format>R8G8B8</format> -->
-        </image>
-        <clip>
-          <near>0.1</near>
-          <far>10.0</far>
-        </clip>
-      </camera>
-      <depth_camera>
-        <output>depth</output>
-      </depth_camera>
-      <topic>/depth_camera</topic>
+      <gz_frame_id>lidar_link</gz_frame_id>
+      <lidar>
+        <scan>
+          <horizontal>
+            <samples>360</samples>
+            <resolution>1.0</resolution>
+            <min_angle>-3.14</min_angle>
+            <max_angle>3.14</max_angle>
+          </horizontal>
+          <vertical>
+            <samples>1</samples>
+            <resolution>0.01</resolution>
+            <min_angle>0</min_angle>
+            <max_angle>0</max_angle>
+          </vertical>
+        </scan>
+        <range>
+          <min>0.2</min>
+          <max>8.0</max>
+          <resolution>0.02</resolution>
+        </range>
+        <noise>
+          <type>gaussian</type>
+          <mean>0.0</mean>
+          <stddev>0.01</stddev>
+        </noise>
+      </lidar>
     </sensor>
   </gazebo>
